File: dao_board.kicad_sch (KiCad schematic)
At the start: 44 parts, among them J1 DISH_LED, J10 KEY6, J11 KEY7, J12 START, J13 SELECT, J14 DISH_SENSOR, J3 SWD, J4 GPIO_EXPANSION, J5 KEY1, J6 KEY2, J7 KEY3, J8 KEY4, J9 KEY5, SW1 RESET, SW2 HX 3x4x2-2P-1.6N, U1 MDBT50Q-1MV2, U2 TLC6C598PWR, U3 TLC6C598PWR

Commit message: 途中まで配線、あとなぜかマイコンにVBUSを接続してなかったので回路図側は修正
Connections:
- net VBUS_5V: now also U1.30 (VDDH), U1.32 (VBUS)
- no-connect marks 37 -> 35
Changed lines of the file:
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@@
-	)
-	(no_connect
-		(at 113.03 80.01)
 	)
 	(no_connect
@@
 	)
 	(no_connect
-		(at 110.49 80.01)
-	)
-	(no_connect
 		(at 130.81 158.75)
 	)
@@
 	(wire
 		(pts
+			(xy 113.03 68.58) (xy 113.03 80.01)
+		)
+		(stroke
+			(width 0)
+			(type default)
+		)
+	)
+	(wire
+		(pts
 			(xy 257.81 93.98) (xy 260.35 93.98)
 		)
@@
 	(wire
 		(pts
+			(xy 110.49 68.58) (xy 110.49 80.01)
+		)
+		(stroke
+			(width 0)
+			(type default)
+		)
+	)
+	(wire
+		(pts
 			(xy 186.69 109.22) (xy 189.23 109.22)
 		)
@@
 			(width 0)
 			(type default)
+		)
+	)
+	(label "VBUS_5V"
+		(at 110.49 68.58 270)
+		(effects
+			(font
+				(size 1.27 1.27)
+			)
+			(justify right bottom)
 		)
 	)
@@
 		(effects
 			(font
+				(size 1.27 1.27)
+			)
+			(justify right bottom)
+		)
+	)
+	(label "VBUS_5V"
+		(at 113.03 68.58 270)
+		(effects
+			(font

Commit message: JLCPCB用にデータを用意中
Parts:
- U1: LCSC Part (none) -> C5118826
Changed lines of the file:
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@@
+			)
+		)
+		(property "LCSC Part" "C5118826"
+			(at 110.49 125.73 0)
+			(hide yes)
+			(show_name no)
+			(do_not_autoplace no)
+			(effects
+				(font
+					(size 1.27 1.27)
+				)
 			)
 		)

Commit message: 問題ないとわかっている違反を除外、一応ライブラリを更新したけどなんかうまく行ってないので除外するしか手段がなかった
Parts:
- U1: footprint RF_Module:Raytac_MDBT50Q -> c5118826:Raytac_MDBT50Q_FIXED
- USBC1: footprint c165948:USB-C_SMD-TYPE-C-31-M-12_1 -> c165948:USB-C_SMD-TYPE-C-31-M-12_1_FIXED
Changed lines of the file:
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@@
 			)
 		)
-		(property "Footprint" "c165948:USB-C_SMD-TYPE-C-31-M-12_1"
+		(property "Footprint" "c165948:USB-C_SMD-TYPE-C-31-M-12_1_FIXED"
 			(at 49.53 62.23 0)
 			(hide yes)
@@
 			)
 		)
-		(property "Footprint" "RF_Module:Raytac_MDBT50Q"
+		(property "Footprint" "c5118826:Raytac_MDBT50Q_FIXED"
 			(at 110.49 130.81 0)
 			(hide yes)
